File: KiCad-actions-test.sch (KiCad schematic (older format))
At the start: 3 parts

Commit message: add pcb design
Parts:
- BT1: footprint (none) -> Battery:BatteryHolder_Keystone_2468_2xAAA
- D1: footprint (none) -> LED_THT:LED_D5.0mm
- R1: footprint (none) -> Resistor_THT:R_Axial_DIN0614_L14.3mm_D5.7mm_P25.40mm_Horizontal
Changed lines of the file:
@@
 F 0 "BT1" H 3508 3746 50  0000 L CNN
 F 1 "AAA Battery x 2" H 3508 3655 50  0000 L CNN
-F 2 "" V 3400 3760 50  0001 C CNN
+F 2 "Battery:BatteryHolder_Keystone_2468_2xAAA" V 3400 3760 50  0001 C CNN
 F 3 "~" V 3400 3760 50  0001 C CNN
 	1    3400 3700
@@
 F 0 "D1" V 4389 3532 50  0000 R CNN
 F 1 "red LED" V 4298 3532 50  0000 R CNN
-F 2 "" H 4350 3650 50  0001 C CNN
+F 2 "LED_THT:LED_D5.0mm" H 4350 3650 50  0001 C CNN
 F 3 "~" H 4350 3650 50  0001 C CNN
 	1    4350 3650
@@
 F 0 "R1" V 3693 3350 50  0000 C CNN
 F 1 "330" V 3784 3350 50  0000 C CNN
-F 2 "" V 3830 3350 50  0001 C CNN
+F 2 "Resistor_THT:R_Axial_DIN0614_L14.3mm_D5.7mm_P25.40mm_Horizontal" V 3830 3350 50  0001 C CNN
 F 3 "~" H 3900 3350 50  0001 C CNN
 	1    3900 3350
